File: schematic/OF_link_CATV_tester/OF_link_CATV_tester-Aleksejsm.kicad_pcb (KiCad board)
At the start: 2 copper layers, 99.9 x 94.5 mm, 122 parts, among them IC1 OPA2320, IC3 ADG904-R, IC4 HMC624, IC5 LT5537, IC6 ADS1219, IC7 SN74CB3Q3251, IC8 SN74CB3Q3251, J1 Conn_01x10, J10 Conn_01x12, J11 Conn_01x12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

Commit message: Updated schematic and PCB
Changed error footprints in PCB
Parts:
- C12: value 33n -> 3.3n
- C4: value ? -> 100n
- IC7, IC8: footprint Package_DFN_QFN:DFN-16-1EP_3x4mm_P0.45mm_EP1.7x3.3mm -> Package_SO:SSOP-16_4.4x5.2mm_P0.65mm
- J4: value Conn_02x4 -> Conn_02x04
- moved R11 3.68 mm to (86.1, 91.1)
- moved IC7 1.80 mm to (93.6, 89.5)
- moved IC8 1.42 mm to (93.6, 98.7)
Routing:
- net +3V3: track 588.3 -> 602.2 mm
- net /S0: track 34.6 -> 28.7 mm
- net /S1: track 38.1 -> 32.9 mm
- net Net-(IC7-Pad2): track 19.7 -> 15.8 mm
- net Net-(IC7-Pad1): track 19.3 -> 15.6 mm, vias 0 -> 2
- net Net-(IC7-Pad15): track 16.2 -> 12.6 mm
- net Net-(IC7-Pad14): track 17.7 -> 14.1 mm
- net Net-(IC7-Pad3): track 19.6 -> 16.3 mm
- net Net-(IC7-Pad4): track 20.3 -> 17.0 mm, vias 2 -> 0
- net Net-(IC7-Pad12): track 20.3 -> 17.4 mm, vias 2 -> 0
- net Net-(IC7-Pad13): track 18.5 -> 16.1 mm, vias 2 -> 0
- net Net-(C1-Pad1): track 16.1 -> 14.1 mm
- net GND: track 304.9 -> 306.6 mm
- net /S2: track 34.9 -> 36.5 mm, vias 2 -> 0
- net Net-(C2-Pad2): track 21.8 -> 20.4 mm
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Other:
- board text added: "12"
- board text added: "12 - RD- 13 - RD+ 18 - TD+ 19 - TD-"
- board text added: "13"
- board text added: "18"
- board text added: "19"
- board text added: "2"
- board text added: "2 - TX_F 3 - TX_D 4 - MD2 5 - MD1"
- board text added: "3"
- board text added: "4"
- board text added: "5"
- board text added: "6"
- board text added: "6 - MD0 7 - Rate 8 - LOS"
- board text added: "7"
- board text added: "8"
