File: schematic/OF_link_CATV_tester/OF_link_CATV_tester-Aleksejsm.sch (KiCad schematic (older format))
At the start: 126 parts, among them IC1 OPA2320, IC3 ADG904-R, IC4 HMC624, IC5 LT5537, IC6 ADS1219, IC7 SN74CB3Q3251, IC8 SN74CB3Q3251, J1 Conn_01x10, J10 Conn_01x12, J11 Conn_01x12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

Commit message: Updated schematic and PCB
Changed error footprints in PCB
Parts:
- C12: value 33n -> 3.3n
- C4: value ? -> 100n
- IC7, IC8: footprint Package_DFN_QFN:DFN-16-1EP_3x4mm_P0.45mm_EP1.7x3.3mm -> Package_SO:SSOP-16_4.4x5.2mm_P0.65mm
- J4: value Conn_02x4 -> Conn_02x04
Connections:
- no-connect marks 4 -> 6
Other:
- note added: "+3.3v Power pins"
- note added: "+5.0v Power pins"
- note added: "4x Photodiode\nCMOS Multiplexer"
- note added: "4x Photodiode\nInput connectors"
- note added: "Active Low Digital Input. \nWhen high, the device is disabled \nand all switches are off. When low, \nAx logic inputs determine On switches."
- note added: "Inputs control the data \npath of the multiplexer"
- note added: "Parallel/Serial Mode Select. \nFor parallel mode operation, \nset this pin to low. \nFor serial mode operation, \nset this pin to high."
- note added: "Power IN\nconnector"
- note added: "Programmable-Gain\nTransimpedance Amplifiers\nFET switching controll"
- note added: "SFP module port\nNr.1"
- note added: "SFP module port\nNr.2"
- note added: "SFP module port\nNr.3"
- note added: "The I2C communication\nDRDY - Data ready, active low."
- moved on the sheet: C1, C10, C11, C12, C13, C14, C15, C16, C17, C18, C19, C2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
